File: Hardware/Shock_board/Shock_board.kicad_pcb (KiCad board)
At the start: 2 copper layers, 212.3 x 88.3 mm, 66 parts, among them P1 220_VAC In, P3 5_VDC In, Q1 BC547, Q2 BC547, Q3 BC547, Q4 BC547, Q5 BC547, Q6 BC547, Q7 BC547, Q8 BC547, U1 PC817, U10 PC817, U11 PC817, U12 PC817, U13 PC817, U14 PC817, U15 PC817, U16 PC817, U17 PC817, U18 PC817, U19 PC817, U2 PC817, U20 PC817, U21 PC817, U22 PC817, U23 PC817, U24 PC817, U3 PC817, U4 PC817, U41 Rectifier_2KBP06M, U5 PC817, U6 PC817, U7 PC817, U8 PC817, U9 PC817

Commit message: update_May_20_2026
Parts:
- Potentiometer: value 500k -> 1M
- R25: value 200k -> 75k
Changed lines of the file:
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@@
 			)
 		)
-		(property "Value" "200k"
+		(property "Value" "75k"
 			(at 5.08 2.31 90)
 			(layer "F.SilkS")
@@
 			)
 		)
-		(property "Value" "500k"
+		(property "Value" "1M"
 			(at -0.762 7.663 90)
 			(layer "F.SilkS")
