File: Hardware/Shock_board/Shock_board.kicad_sch (KiCad schematic)
At the start: 9 parts, among them J3 Conn_01x04_Pin, J4 Conn_02x08_Odd_Even, J5 Conn_01x04_Pin, P1 220VAC In, P3 5VDC In, U41 Rectifier_2KBP06M

Commit message: update_May_20_2026
Parts:
- R25: value 200k -> 75k
- RV1: value 500k -> 1M
Other:
- note added: "450V"
- note removed: "350V"
- note removed: "Conditioning Chamber"
- title: (none) -> Shock Control Board
- moved on the sheet: J4
